File: Hat Version 2.0/HAT_CM4V2.1/CM4-Batteries.kicad_sch (KiCad schematic)
At the start: 5 parts

Commit message: Updated to second protype release
Connections:
- net BATT+ renamed BAT+
Changed lines of the file:
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@@
   (title_block
     (title "ConnectBox CM4 for China Case")
-    (date "2022-04-07")
-    (rev "1.8.3")
+    (date "2022-03-18")
+    (rev "1.8.2")
     (comment 1 "JRA")
   )
@@
     (effects (font (size 1.524 1.524)) (justify right))
   )
-  (hierarchical_label "BATT+" (shape output) (at 119.38 74.93 180)
+  (hierarchical_label "BAT+" (shape output) (at 119.38 74.93 180)
     (effects (font (size 1.524 1.524)) (justify right))
   )
