File: Hat Version 2.0/HAT_CM4V2.1/CM4_BattBoard-Battery.kicad_sch (KiCad schematic)
At the start: 53 parts, among them Q1 2N7002, Q10 3J15, Q11 3J15, Q12 3J15, Q13 8205A, Q14 3J15, Q15 3J15, Q16 3J15, Q17 8205A, Q2 3J15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

Commit message: Updated to second protype release
Parts:
- removed LED12: Blue, LED_SMD:LED_0603_1608Metric, symbol Device:LED_Small
- removed R57: 1K, Resistor_SMD:R_0603_1608Metric, symbol Device:R
- added D1, D2: MMBD914, Diode_SMD:D_SOT-23_ANK, symbol Diode:1N914
- added U2: 74LVCE1G126, Package_TO_SOT_SMD:SOT-23-5, symbol Custom_1:74LVCE1G126
- Q10, Q14, Q2, Q6: symbol Custom_1:Q_PMOS_GSD -> Device:Q_PMOS_GSD
- Q11, Q12, Q15, Q16, Q3, Q4, Q7, Q8: symbol Custom_1:Q_PMOS_GSD -> CustomComponents:Q_PMOS_GSD
- R2: value 20K -> 2.2K; DigiKey P/N 311-20.0KHRCT-ND -> 311-2.20KHRCT-ND; Manufacturer P/N RC0603FR-0720KL -> RC0603FR-072K2L
- U1: symbol Custom_1:ATtiny88-AU -> MCU_Microchip_ATtiny:ATtiny88-AU
Connections:
- net AC_IN: now also D2.2 (A)
- net PWR_GND: now also U2.3 (Gnd); no longer R12.2, R18.2, R2.2, R24.2, R6.2, U1.21 (GND), U1.5 (GND)
- net /BT1_ENA: now also U2.2 (A)
- net /BT1_ENA_B: now also U2.4 (Y)
- net ADC2: now reaches R1.1, R2.1, U1.25 (PC2)
- net at Q1.1 (G), R3.2, R4.2: now also U2.1 (OE)
- net ADC0: now reaches U1.23 (PC0)
- net ADC1: now reaches U1.24 (PC1)
- net +5V renamed 5V
- net 5V: now also D1.2 (A)
- net 5V_OVR: no longer names the net of U1.10 (PD6)
- net AXP_EXTEN: no longer names the net of U1.2 (PD4)
- net BATT+ renamed BAT+
- net BAT+: now also U2.5 (Vcc); no longer U1.18 (AVCC), U1.4 (VCC)
- net HEARTBEAT renamed ADC3
- net PB_IN: no longer names the net of U1.11 (PD7)
- net PWR_IRQ: no longer names the net of U1.9 (PD5)
- new net: R12.2, R18.2, R2.2, R24.2, R6.2, U1.21 (GND), U1.5 (GND)
- new net: D1.1 (K), D2.1 (K), U1.18 (AVCC), U1.4 (VCC)
- no-connect marks 16 -> 18
Other:
- note added: "FUTURE (?): Remove Batt Reversed LEDs since there is no battery board on which to mount them. For the moment, leave battery selected leds in place (debug)"
- note added: "This circuit is the same as the reworked battery board using rev 1.7.4 boards - 01/24/22 (except R6, 13, 20, 27 were tied to PWR_GND and buffer U15 has been added) - Isolated ATTiny gnd and resistors R6, 13, 20, 27 and added JP1 to allow easy select of whether they are tied to PWR_GND or switched gnd"
- note removed: "ATTiny needs to sense for AC_IN, but since the ATTiny is controlling the 5V supply via PWR_CTL, it does not need a sense to see when it is on"
- note removed: "Logic: We will control power ON from AXP209: - (control from ATTiny opens possibility of bricking the unit if ATTiny not programmed correctly) - Power on at either PB or AC_IN - Power off signal from AXP209 initiates power down but final time from ATTiny Role of ATTiny: Generally, the ATTiny will be used to override the power control state of the AXP209 when: a) AXP209 calls for power on in respo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"
- moved on the sheet: Q1, Q10, Q14, Q2, Q6, R1, R2, R3, R4, U1
