File: Hat Version 2.0/HAT_CM4V2.1/HAT_CM4-CM4-GPIO.kicad_sch (KiCad schematic)
At the start: 26 parts, among them J1 Micro_SD_Card, J6 MagJack-S811, P1 Conn_01x04, U5 TPD4EUSB30, U6 RT9742ANGJ5F

Commit message: Updated to second protype release
Parts:
- added C11: 10uF, Capacitor_SMD:C_0603_1608Metric, symbol Device:C
- added LED9: Blue, LED_SMD:LED_0603_1608Metric, symbol Device:LED_Small
- added R56: 510, Resistor_SMD:R_0603_1608Metric, symbol Device:R
- LED7: value Blue -> Amber; DigiKey P/N 1830-1068-1-ND -> 160-1445-1-ND; Manufacturer Inolux -> Lite-On Inc.; Manufacturer P/N IN-S63BT5B -> LTST-C191KFKT
- PB1, PB2: symbol Custom_1:SPST-PUSH -> CustomComponents:SPST-PUSH
- R42: value 10K -> 51K; DigiKey P/N 311-10.0KHRCT-ND -> 311-51.0KHRCT-ND; Manufacturer P/N RC0603FR-0710KL -> RC0603FR-071KL
- R43: value 33K -> 1K; DigiKey P/N 311-33.0KHRCT-ND -> 311-1.00KHRCT-ND; Manufacturer P/N RC0603FR-0733KL -> RC0603FR-071KL
Connections:
- net PWR_IRQ is gone; now on net +3.3v: R42.1
- net +3.3v: now also R56.1
- net GND: now also C11.2; no longer R43.1
- net GPIO19: now also LED9.1 (K)
- net GPIO_IRQ: now also R43.1, C11.1; no longer R42.2, R43.2
- net PB_IN renamed PowerSwitch
- new net: LED9.2 (A), R56.2
- new net EXT_ENA: R42.2, R43.2
Other:
- moved on the sheet: R42, R43
