File: Hat Version 2.0/HAT_CM4V2.1/HAT_CM4-CM4-HS.kicad_sch (KiCad schematic)
At the start: 6 parts, among them J2 690-019-298-412, U9 RT9742ANGJ5F

Commit message: Updated to second protype release
Connections:
- net USBOTG_ID: now reaches Module1.101 (USB_OTG_ID)
- no-connect marks 5 -> 4
Changed lines of the file:
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@@
   (title_block
     (title "ConnectBox CM4 for China Case")
-    (date "2022-04-07")
-    (rev "1.8.3")
+    (date "2022-03-18")
+    (rev "1.8.2")
     (comment 1 "JRA")
   )
@@
   (no_connect (at 85.09 60.96))
   (no_connect (at 248.92 171.45))
-  (no_connect (at 152.4 55.88))
   (no_connect (at 85.09 58.42))
   (no_connect (at 243.84 204.47))
@@
     (effects (font (size 1.27 1.27)) (justify left))
   )
+  (hierarchical_label "USBOTG_ID" (shape input) (at 152.4 55.88 0)
+    (effects (font (size 1.27 1.27)) (justify left))
+  )
