File: Hat Version 2.0/HAT_CM4V2.1/HAT_CM4-Charge.kicad_sch (KiCad schematic)
At the start: 21 parts, among them U3 AXP209

Commit message: Updated to second protype release
Connections:
- net AXP_EXTEN renamed EXT_EN
- net BATT+ renamed BAT+
- net PB_IN renamed PowerSwitch
Changed lines of the file:
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@@
   (title_block
     (title "ConnectBox CM4 for China Case")
-    (date "2022-04-07")
-    (rev "1.8.3")
+    (date "2022-03-18")
+    (rev "1.8.2")
     (comment 1 "JRA")
   )
@@
     (stroke (width 0) (type solid) (color 0 0 0 0))
   )
+  (wire (pts (xy 261.62 97.79) (xy 342.9 97.79))
+    (stroke (width 0) (type solid) (color 0 0 0 0))
+  )
   (wire (pts (xy 207.01 111.76) (xy 207.01 109.22))
     (stroke (width 0) (type solid) (color 0 0 0 0))
@@
     (stroke (width 0) (type solid) (color 0 0 0 0))
   )
-  (wire (pts (xy 215.9 116.84) (xy 96.52 116.84))
+  (wire (pts (xy 215.9 116.84) (xy 102.235 116.84))
     (stroke (width 0) (type solid) (color 0 0 0 0))
   )
@@
     (stroke (width 0) (type solid) (color 0 0 0 0))
   )
-  (wire (pts (xy 261.62 97.79) (xy 340.995 97.79))
-    (stroke (width 0) (type default) (color 0 0 0 0))
-  )
   (wire (pts (xy 290.83 177.8) (xy 341.63 177.8))
     (stroke (width 0) (type solid) (color 0 0 0 0))
@@
     (stroke (width 0) (type solid) (color 0 0 0 0))
   )
-  (label "BATT+" (at 149.86 83.82 0)
+  (label "A_GND" (at 285.75 74.93 0)
+    (effects (font (size 1.524 1.524)) (justify left bottom))
+  )
+  (label "BAT+" (at 149.86 83.82 0)
     (effects (font (size 1.524 1.524)) (justify left bottom))
   )
@@
     (effects (font (size 1.778 1.778)) (justify left))
   )
-  (hierarchical_label "PB_IN" (shape input) (at 96.52 116.84 180)
+  (hierarchical_label "PowerSwitch" (shape input) (at 102.235 116.84 180)
     (effects (font (size 1.778 1.778)) (justify right))
   )
@@
     (effects (font (size 1.778 1.778)) (justify left))
   )
-  (hierarchical_label "AXP_EXTEN" (shape output) (at 340.995 97.79 0)
-    (effects (font (size 1.524 1.524)) (justify left))
+  (hierarchical_label "EXT_EN" (shape output) (at 342.9 97.79 0)
+    (effects (font (size 1.778 1.778)) (justify left))
   )
   (hierarchical_label "IPS_OUT" (shape output) (at 341.63 66.04 0)
@@
     (effects (font (size 1.778 1.778)) (justify right))
   )
-  (hierarchical_label "BATT+" (shape input) (at 96.52 96.52 180)
+  (hierarchical_label "BAT+" (shape input) (at 96.52 96.52 180)
     (effects (font (size 1.778 1.778)) (justify right))
   )
@@
       (effects (font (size 1.27 1.27)) hide)
     )
-    (property "Datasheet" "~" (id 3) (at 299.72 140.97 90))
+    (property "Datasheet" "" (id 3) (at 299.72 140.97 90))
     (property "Manufacturer" "Lite-On Inc." (id 4) (at 299.72 140.97 90)
       (effects (font (size 1.524 1.524)) hide)
