File: Hat Version 2.0/HAT_CM4V2.1/HAT_CM4-Power.kicad_sch (KiCad schematic)
At the start: 20 parts, among them U7 AP22814A, U8 MAX1709ESE

Commit message: Updated to second protype release
Parts:
- removed D1: MMBD914, Diode_SMD:D_SOT-23_ANK, symbol Diode:1N914
- removed R50: 20K, Resistor_SMD:R_0603_1608Metric, symbol Device:R
- added C13: 22uF, Capacitor_SMD:C_0603_1608Metric, symbol Device:C
- added D4, D6: MMBD914, Diode_SMD:D_SOT-23_ANK, symbol Diode:1N914
- C14, C15, C19, C20: symbol Custom_1:CP -> Device:CP
- L2: footprint Inductor_SMD:L_Taiyo-Yuden_NR-50xx -> Inductor_SMD:L_Taiyo-Yuden_MD-5050; symbol Custom_1:INDUCTOR-1 -> CustomComponents:INDUCTOR-1; DigiKey P/N 587-2404-1-ND -> 490-16290-1-ND - Cut Tape (CT); Manufacturer Taiyo Yuden -> Murata; Manufacturer P/N NRS5020T1R5NMGJ -> LQH5BPN1R0N38L
- L3: symbol Custom_1:INDUCTOR-1 -> CustomComponents:INDUCTOR-1
- R44: value 100K -> 1M; DigiKey P/N 311-100KHRCT-ND -> 311-1.00MHRCT-ND; Manufacturer P/N RC0603FR-07100KL -> RC0603FR-071ML
- U7: symbol Custom_1:AP22814A -> CustomComponents:AP22814A
Connections:
- net PWR_GND: now also C13.2
- net 5V_OVR renamed SNS_EN
- net SNS_EN: now also C13.1, D4.1 (K), D6.1 (K)
- new net EXT_EN: D4.2 (A)
- new net OVR_EN: D6.2 (A)
Other:
- note removed: "AXP_EXTEN from AXP209 to control power on. 5V_OVR from ATTiny88 used to override power up (if not initiated by pushbutton) and power down (to extend power down time)."
