File: Hat Version 2.0/HAT_CM4V2.1/HAT_CM4-USB_Hub.kicad_sch (KiCad schematic)
At the start: 31 parts, among them J3 USB_A, J4 USB_A, J5 USB-C, J7 Flex-4, U12 RT9742ANGJ5F, U13 USB2514B-I/M2, U15 HC-R8812AF1, Y1 24MHz

Commit message: Updated to second protype release
Parts:
- removed J7: Flex-4, CustomComponents:SFW4R-1, symbol Custom_1:Flex-4
- C30: footprint Capacitor_SMD:CP_Elec_5x3 -> Capacitor_SMD:CP_Elec_6.3x4.5; symbol Custom_1:CP -> Device:CP; DigiKey P/N 565-4332-1-ND -> 493-3819-1-ND; Manufacturer Nippon Chemi-Con -> Nichicon; Manufacturer P/N APXF6R3ARA151ME61G -> RSL0J101MCN1GB
Other:
- note added: "OTG"
- note removed: "Optional Flex connector (USB port)"
Changed lines of the file:
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@@
   (title_block
     (title "ConnectBox CM4 for China Case")
-    (date "2022-04-07")
-    (rev "1.8.3")
+    (date "2022-03-18")
+    (rev "1.8.2")
     (comment 1 "JRA")
   )
@@
     (stroke (width 0) (type solid) (color 0 0 0 0))
   )
+  (wire (pts (xy 204.47 113.03) (xy 213.36 113.03))
+    (stroke (width 0) (type solid) (color 0 0 0 0))
+  )
   (wire (pts (xy 181.61 92.71) (xy 181.61 95.25))
     (stroke (width 0) (type solid) (color 0 0 0 0))
   )
-  (wire (pts (xy 204.47 113.03) (xy 237.49 113.03))
-    (stroke (width 0) (type default) (color 0 0 0 0))
-  )
   (wire (pts (xy 302.895 65.405) (xy 314.325 65.405))
     (stroke (width 0) (type solid) (color 0 0 0 0))
@@
   (wire (pts (xy 322.58 201.93) (xy 306.07 201.93))
     (stroke (width 0) (type solid) (color 0 0 0 0))
-  )
-  (wire (pts (xy 237.49 115.57) (xy 233.68 115.57))
-    (stroke (width 0) (type default) (color 0 0 0 0))
   )
   (wire (pts (xy 334.01 153.67) (xy 336.55 153.67))
@@
     (stroke (width 0) (type default) (color 0 0 0 0))
   )
-  (wire (pts (xy 229.87 107.95) (xy 237.49 107.95))
-    (stroke (width 0) (type default) (color 0 0 0 0))
-  )
-  (wire (pts (xy 204.47 110.49) (xy 237.49 110.49))
+  (wire (pts (xy 204.47 110.49) (xy 213.36 110.49))
     (stroke (width 0) (type solid) (color 0 0 0 0))
   )
@@
   (wire (pts (xy 109.855 142.24) (xy 109.855 147.32))
     (stroke (width 0) (type solid) (color 0 0 0 0))
-  )
-  (wire (pts (xy 233.68 115.57) (xy 233.68 119.38))
-    (stroke (width 0) (type default) (color 0 0 0 0))
   )
   (wire (pts (xy 168.91 92.71) (xy 168.91 95.25))
@@
     (effects (font (size 1.778 1.778)) (justify left bottom))
   )
-  (text "Optional Flex connector\n(USB port)" (at 252.73 113.03 0)
-    (effects (font (size 1.27 1.27)) (justify left bottom))
-  )
   (text "USB 2.0 Hub" (at 205.5368 93.9292 180)
+    (effects (font (size 1.27 1.27)) (justify right bottom))
+  )
+  (text "OTG" (at 325.755 52.705 180)
     (effects (font (size 1.27 1.27)) (justify right bottom))
   )
@@
   )
   (label "nOCS1" (at 213.36 118.11 180)
-    (effects (font (size 1.27 1.27)) (justify right bottom))
-  )
-  (label "VBUS" (at 229.87 107.95 180)
     (effects (font (size 1.27 1.27)) (justify right bottom))
   )
@@
     (pin "1")
   )
-  (symbol (lib_name "GND_2") (lib_id "power:GND") (at 242.57 156.21 0) (unit 1)
+  (symbol (lib_id "power:GND") (at 242.57 156.21 0) (unit 1)
     (in_bom yes) (on_board yes)
     (property "Reference" "#PWR037" (id 0) (at 242.57 162.56 0)
@@
     (pin "1")
     (pin "2")
-  )
-  (symbol (lib_id "Custom_1:Flex-4") (at 240.03 111.76 0) (unit 1)
-    (in_bom yes) (on_board yes) (fields_autoplaced)
-    (property "Reference" "J7" (id 0) (at 247.0912 112.239 0)
-      (effects (font (size 1.27 1.27)) (justify left))
-    )
-    (property "Value" "Flex-4" (id 1) (at 234.95 119.38 0)
-      (effects (font (size 1.27 1.27)) hide)
-    )
-    (property "Footprint" "CustomComponents:SFW4R-1" (id 2) (at 238.76 128.905 0)
-      (effects (font (size 1.27 1.27)) hide)
-    )
-    (property "Datasheet" "" (id 3) (at 240.03 111.76 0)
-      (effects (font (size 1.27 1.27)) hide)
-    )
-    (property "Manufacturer" "Amphenol" (id 4) (at 229.87 127 0)
-      (effects (font (size 1.27 1.27)) hide)
-    )
-    (property "Manufacturer P/N" "SFW4R" (id 5) (at 240.03 127 0)
-      (effects (font (size 1.27 1.27)) hide)
-    )
-    (property "Description" "Connector FFC Bottom 4 Position 1.00mm R/A" (id 6) (at 242.57 123.19 0)
-      (effects (font (size 1.27 1.27)) hide)
-    )
-    (property "DigiKey P/N" "609-SFW4R-1STE1HLFCT-ND" (id 7) (at 239.395 125.095 0)
-      (effects (font (size 1.27 1.27)) hide)
-    )
-    (pin "1")
-    (pin "2")
-    (pin "3")
-    (pin "4")
   )
   (symbol (lib_id "Device:C") (at 152.4 76.2 0) (unit 1)
@@
     (pin "1")
   )
-  (symbol (lib_id "Custom_1:CP") (at 189.23 210.82 0) (unit 1)
+  (symbol (lib_id "Device:CP") (at 189.23 210.82 0) (unit 1)
     (in_bom yes) (on_board yes)
     (property "Reference" "C30" (id 0) (at 192.2272 209.677 0)
@@
       (effects (font (size 1.27 1.27)) (justify left))
     )
-    (property "Footprint" "Capacitor_SMD:CP_Elec_5x3" (id 2) (at 190.1952 214.63 0)
+    (property "Footprint" "Capacitor_SMD:CP_Elec_6.3x4.5" (id 2) (at 190.1952 214.63 0)
       (effects (font (size 1.27 1.27)) hide)
     )
@@
       (effects (font (size 1.27 1.27)) hide)
     )
-    (property "Manufacturer" "Nippon Chemi-Con" (id 4) (at 189.23 210.82 0)
-      (effects (font (size 1.778 1.778)) hide)
-    )
-    (property "Manufacturer P/N" "APXF6R3ARA151ME61G" (id 5) (at 189.23 210.82 0)
-      (effects (font (size 1.778 1.778)) hide)
-    )
-    (property "Description" "150uf, 6.3V Alum Polymer Cap" (id 6) (at 189.23 210.82 0)
-      (effects (font (size 1.778 1.778)) hide)
-    )
-    (property "DigiKey P/N" "565-4332-1-ND" (id 7) (at 189.23 210.82 0)
+    (property "Manufacturer" "Nichicon" (id 4) (at 189.23 210.82 0)
+      (effects (font (size 1.27 1.27)) hide)
+    )
+    (property "Manufacturer P/N" "RSL0J101MCN1GB" (id 5) (at 189.23 210.82 0)
+      (effects (font (size 1.27 1.27)) hide)
+    )
+    (property "Description" "Capacitor, SP-Cap, 100u, 6.3V, 18mR ESR" (id 6) (at 189.23 210.82 0)
+      (effects (font (size 1.27 1.27)) hide)
+    )
+    (property "DigiKey P/N" "493-3819-1-ND" (id 7) (at 189.23 210.82 0)
       (effects (font (size 1.778 1.778)) hide)
     )
@@
       (effects (font (size 1.27 1.27)) hide)
     )
-    (pin "1")
-  )
-  (symbol (lib_name "GND_1") (lib_id "power:GND") (at 233.68 119.38 0) (unit 1)
-    (in_bom yes) (on_board yes)
-    (property "Reference" "#PWR019" (id 0) (at 233.68 125.73 0)
-      (effects (font (size 1.27 1.27)) hide)
-    )
-    (property "Value" "GND" (id 1) (at 233.807 123.7742 0))
-    (property "Footprint" "" (id 2) (at 233.68 119.38 0)
-      (effects (font (size 1.27 1.27)) hide)
-    )
-    (property "Datasheet" "" (id 3) (at 233.68 119.38 0)
-      (effects (font (size 1.27 1.27)) hide)
-    )
