File: Hat Version 2.0/HAT_CM4V2.1/HAT_CM4_182.kicad_sch (KiCad schematic)
At the start: 3 parts

Commit message: Updated to second protype release
Other:
- sheet Batteries ports: added BAT+; removed BATT+
- sheet Battery ports: added 5V, BAT+; removed +5V, 5V_OVR, AXP_EXTEN, BATT+, PB_IN, PWR_IRQ
- sheet CM4_GPIO ports: added EXT_ENA, PowerSwitch; removed PB_IN, PWR_IRQ
- sheet CM4_HighSpeed ports: added USBOTG_ID; removed none
- sheet Charger ports: added BAT+, EXT_EN, PowerSwitch; removed AXP_EXTEN, BATT+, PB_IN
- sheet Power ports: added EXT_EN; removed 5V_OVR, AXP_EXTEN
- sheet USB Hub ports: added USBOTG; removed none
